File: protoboard/_autosave-ClearGauntlet.kicad_pcb (KiCad board)
At the start: 2 copper layers, 66 x 55.9 mm, 21 parts

Commit message: Check autosaves
Parts:
- removed the REF** at (203.2, 81.3)
- removed the REF** at (215.9, 96.5)
- removed the REF** at (210.8, 78.7)
- removed the REF** at (172.8, 104.1)
- removed the REF** at (221.0, 114.3)
- removed the REF** at (183.0, 114.3)
- removed the REF** at (228.6, 81.3)
- removed the REF** at (210.8, 111.8)
- removed the REF** at (218.4, 94.0)
- removed the REF** at (172.8, 88.9)
- removed the REF** at (213.4, 83.8)
- removed the REF** at (172.8, 99.1)
- removed the REF** at (182.9, 99.1)
- removed the REF** at (182.9, 109.2)
- removed the REF** at (182.9, 104.1)
- removed the REF** at (172.8, 109.2)
- removed the REF** at (172.8, 94.0)
- removed the REF** at (182.9, 94.0)
- added REF**: PinHeader_1x03_P2.54mm_Vertical, Connector_PinHeader_2.54mm:PinHeader_1x03_P2.54mm_Vertical, F.Cu at (182.9, 109.2)
- added REF**: PinHeader_1x03_P2.54mm_Vertical, Connector_PinHeader_2.54mm:PinHeader_1x03_P2.54mm_Vertical, F.Cu at (182.9, 99.1)
- added REF**: PinHeader_1x03_P2.54mm_Vertical, Connector_PinHeader_2.54mm:PinHeader_1x03_P2.54mm_Vertical, F.Cu at (182.9, 96.5)
- added REF**: PinHeader_1x03_P2.54mm_Vertical, Connector_PinHeader_2.54mm:PinHeader_1x03_P2.54mm_Vertical, F.Cu at (172.7, 99.1)
- added REF**: PinHeader_1x03_P2.54mm_Vertical, Connector_PinHeader_2.54mm:PinHeader_1x03_P2.54mm_Vertical, F.Cu at (182.9, 111.8)
- added REF**: PinHeader_1x03_P2.54mm_Vertical, Connector_PinHeader_2.54mm:PinHeader_1x03_P2.54mm_Vertical, F.Cu at (172.7, 109.2)
- added REF**: PinHeader_1x03_P2.54mm_Vertical, Connector_PinHeader_2.54mm:PinHeader_1x03_P2.54mm_Vertical, F.Cu at (172.7, 106.7)
- added REF**: PinHeader_1x03_P2.54mm_Vertical, Connector_PinHeader_2.54mm:PinHeader_1x03_P2.54mm_Vertical, F.Cu at (172.7, 101.6)
- added REF**: PinHeader_1x03_P2.54mm_Vertical, Connector_PinHeader_2.54mm:PinHeader_1x03_P2.54mm_Vertical, F.Cu at (182.9, 94.0)
- added REF**: PinHeader_1x03_P2.54mm_Vertical, Connector_PinHeader_2.54mm:PinHeader_1x03_P2.54mm_Vertical, F.Cu at (182.9, 106.7)
- added REF**: PinHeader_1x03_P2.54mm_Vertical, Connector_PinHeader_2.54mm:PinHeader_1x03_P2.54mm_Vertical, F.Cu at (182.9, 91.4)
- added REF**: PinHeader_1x03_P2.54mm_Vertical, Connector_PinHeader_2.54mm:PinHeader_1x03_P2.54mm_Vertical, F.Cu at (182.9, 104.1)
- added REF**: PinHeader_1x03_P2.54mm_Vertical, Connector_PinHeader_2.54mm:PinHeader_1x03_P2.54mm_Vertical, F.Cu at (182.8, 114.2)
- added REF**: PinHeader_1x03_P2.54mm_Vertical, Connector_PinHeader_2.54mm:PinHeader_1x03_P2.54mm_Vertical, F.Cu at (172.7, 104.1)
- added REF**: PinHeader_1x03_P2.54mm_Vertical, Connector_PinHeader_2.54mm:PinHeader_1x03_P2.54mm_Vertical, F.Cu at (182.9, 101.6)
Routing:
- net (no net): track 240.3 -> 0.00 mm
Other:
- board size 66 x 55.9 mm -> 30.5 x 53.3 mm
