File: v3/lower_v3/lower_v3.kicad_pcb (KiCad board)
At the start: 2 copper layers, 38.1 x 71.1 mm, 4 parts, among them J1 Conn_01x09_MountingPin, J2 Conn_01x09_MountingPin, J4 Conn_01x02_Male, U1 ESP32-DEVKIT-V1

Commit message: Updates
Parts:
- added N1: Housing, Filter:Filter_1109-5_1.1x0.9mm, F.Cu at (170.2, 68.6)
Routing:
- net Net-(J1-Pad9): track 50.4 -> 53.0 mm
Changed lines of the file:
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@@
+    )
+  )
+  (footprint "Filter:Filter_1109-5_1.1x0.9mm" (layer "F.Cu")
+    (at 170.18 68.58)
+    (descr "5-pin SAW filter package - 1.1x0.9 mm Body; (see https://www.murata.com/~/media/webrenewal/support/library/catalog/products/filter/rf/p73e.ashx?la=en-gb)")
+    (tags "Filter 5")
+    (property "Sheetfile" "lower_v3.kicad_sch")
+    (property "Sheetname" "")
+    (attr smd)
+    (fp_text reference "N1" (at 0 1.6) (layer "F.SilkS")
+      (effects (font (size 1 1) (thickness 0.15)))
+    )
+    (fp_text value "Housing" (at 0 -1.4) (layer "F.Fab")
+      (effects (font (size 1 1) (thickness 0.15)))
+    )
+    (fp_text user "${REFERENCE}" (at 0 -2.7) (layer "F.Fab")
+      (effects (font (size 1 1) (thickness 0.15)))
+    )
+    (fp_line (start -0.6 -0.5) (end -0.6 0.5) (layer "F.SilkS") (width 0.12))
+    (fp_line (start 0.6 -0.5) (end -0.6 -0.5) (layer "F.SilkS") (width 0.12))
+    (fp_line (start -0.75 -0.5) (end -0.75 0.5) (layer "F.SilkS") (width 0.12))
+    (fp_line (start -0.6 0.5) (end 0.6 0.5) (layer "F.SilkS") (width 0.12))
+    (fp_line (start 0.6 0.5) (end 0.6 -0.5) (layer "F.SilkS") (width 0.12))
+    (fp_line (start -0.7 -0.6) (end 0.7 -0.6) (layer "F.CrtYd") (width 0.05))
+    (fp_line (start 0.7 0.6) (end -0.7 0.6) (layer "F.CrtYd") (width 0.05))
+    (fp_line (start 0.7 -0.6) (end 0.7 0.6) (layer "F.CrtYd") (width 0.05))
+    (fp_line (start -0.7 0.6) (end -0.7 -0.6) (layer "F.CrtYd") (width 0.05))
+    (fp_line (start -0.55 0.15) (end -0.55 0.45) (layer "F.Fab") (width 0.1))
+    (fp_line (start 0.55 0.45) (end -0.55 0.45) (layer "F.Fab") (width 0.1))
+    (fp_line (start -0.4 0) (end -0.55 0.15) (layer "F.Fab") (width 0.1))
+    (fp_line (start -0.55 -0.15) (end -0.4 0) (layer "F.Fab") (width 0.1))
+    (fp_line (start -0.55 -0.45) (end -0.55 -0.15) (layer "F.Fab") (width 0.1))
+    (fp_line (start 0.55 -0.45) (end 0.55 0.45) (layer "F.Fab") (width 0.1))
+    (fp_line (start -0.55 -0.45) (end 0.55 -0.45) (layer "F.Fab") (width 0.1))
+    (pad "1" smd rect (at -0.385 0 90) (size 0.25 0.18) (layers "F.Cu" "F.Paste" "F.Mask"))
+    (pad "2" smd rect (at 0 0.25 90) (size 0.25 0.18) (layers "F.Cu" "F.Paste" "F.Mask"))
+    (pad "3" smd rect (at 0.385 0.25 90) (size 0.25 0.18) (layers "F.Cu" "F.Paste" "F.Mask"))
+    (pad "4" smd rect (at 0.385 -0.25 90) (size 0.25 0.18) (layers "F.Cu" "F.Paste" "F.Mask"))
+    (pad "5" smd rect (at 0 -0.25 90) (size 0.25 0.18) (layers "F.Cu" "F.Paste" "F.Mask"))
+    (model "${KICAD6_3DMODEL_DIR}/Filter.3dshapes/Filter_1109-5_1.1x0.9mm.wrl" hide
+      (offset (xyz 60 -55 0))
+      (scale (xyz 1 1 1))
+      (rotate (xyz 0 0 0))
+    )
+    (model "C:/Users/Long Nguyen/Documents/RIT/RIT_Fall_22/MSD/ClearGauntlet-PCB/v3/upper_v3/upper_v3_2.step"
+      (offset (xyz -154.5 69 7.5))
+      (scale (xyz 1 1 1))
+      (rotate (xyz 0 0 0))
     )
   )
@@
   (segment (start 160.02 93.705) (end 167.64 86.085) (width 0.25) (layer "B.Cu") (net 9))
   (segment (start 170.18 124.46) (end 170.18 81.28) (width 0.25) (layer "B.Cu") (net 10))
+  (segment (start 169.905 81.005) (end 170.18 81.28) (width 0.25) (layer "B.Cu") (net 10))
   (segment (start 165.1 129.54) (end 170.18 124.46) (width 0.25) (layer "B.Cu") (net 10))
+  (segment (start 167.64 81.005) (end 169.905 81.005) (width 0.25) (layer "B.Cu") (net 10))
   (segment (start 137.435 78.74) (end 142.24 83.545) (width 0.25) (layer "B.Cu") (net 11))
   (segment (start 137.16 78.74) (end 137.435 78.74) (width 0.25) (layer "B.Cu") (net 11))

Commit message: Complete Toast PCB
Parts:
- added J3: Conn_01x21, Connector_PinHeader_2.54mm:PinHeader_1x21_P2.54mm_Horizontal, F.Cu at (150.6, 78.7)
- J1, J2: value Conn_01x09_MountingPin -> Conn_01x05_Male; footprint Connector_PinSocket_2.54mm:PinSocket_1x09_P2.54mm_Vertical -> Connector_PinHeader_2.54mm:PinHeader_1x05_P2.54mm_Vertical
- moved N1 52.8 mm to (118.1, 77.5)
- moved J2 31.4 mm to (135.9, 77.5)
- moved U1 26.2 mm to (130.8, 106.7)
- moved J1 20.1 mm to (125.7, 135.9)
- moved J4 7.73 mm to (144.8, 77.5), turned to -90 degrees
Connections:
- J1 pad 5: Net-(J1-Pad5) -> Net-(U1-Pad30)
- J2 pad 2: Net-(J2-Pad2) -> Net-(U1-Pad28)
- J2 pad 3: Net-(J2-Pad3) -> Net-(U1-Pad27)
- J2 pad 4: Net-(J2-Pad4) -> Net-(U1-Pad5)
- J2 pad 5: Net-(J2-Pad5) -> Net-(U1-Pad4)
- J4 pad 1: GND -> Net-(J4-Pad1)
- J4 pad 2: Net-(J2-Pad9) -> GND
- U1 pad 19: Net-(J2-Pad8) -> Net-(U1-Pad19)
- U1 pad 20: Net-(J2-Pad7) -> Net-(U1-Pad20)
- U1 pad 21: Net-(J2-Pad6) -> Net-(U1-Pad21)
- U1 pad 22: Net-(J2-Pad5) -> Net-(U1-Pad22)
- U1 pad 23: Net-(J2-Pad4) -> Net-(U1-Pad23)
- U1 pad 25: Net-(J2-Pad3) -> Net-(U1-Pad25)
- U1 pad 26: Net-(J2-Pad2) -> Net-(U1-Pad26)
- U1 pad 27: Net-(J1-Pad8) -> Net-(U1-Pad27)
- U1 pad 28: Net-(J1-Pad7) -> Net-(U1-Pad28)
- U1 pad 30: Net-(J1-Pad9) -> Net-(U1-Pad30)
- U1 pad 4: Net-(J1-Pad6) -> Net-(U1-Pad4)
- U1 pad 5: Net-(J1-Pad5) -> Net-(U1-Pad5)
Routing:
- net GND: track 51.0 -> 149.5 mm
- net Net-(J4-Pad1): track 0.00 -> 83.0 mm
- net Net-(J1-Pad9): track 53.0 -> 0.00 mm
- net Net-(J2-Pad8): track 51.3 -> 0.00 mm
- net Net-(U1-Pad30): track 0.00 -> 47.9 mm
- net Net-(J2-Pad7): track 47.7 -> 0.00 mm
- net Net-(J1-Pad6): track 47.2 -> 0.00 mm
- net Net-(J1-Pad7): track 46.6 -> 0.00 mm
- net Net-(J2-Pad6): track 44.1 -> 0.00 mm
- net Net-(J1-Pad5): track 43.6 -> 0.00 mm
- net Net-(J1-Pad8): track 43.0 -> 0.00 mm
- net Net-(J2-Pad5): track 40.5 -> 0.00 mm
- net Net-(J2-Pad4): track 36.9 -> 0.00 mm
- net Net-(J2-Pad3): track 30.8 -> 0.00 mm
- net Net-(U1-Pad5): track 0.00 -> 28.1 mm
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- added copper zone on B.Cu, net GND
- added copper zone on F.Cu, net GND
Other:
- board size 38.1 x 71.1 mm -> 40.6 x 64.8 mm
- board text added: "ClearGauntlet"
