File: joycon-board/joycon/joycon/_autosave-joycon.kicad_pcb (KiCad board)
At the start: 2 copper layers, 21.6 x 20 mm, 11 parts, among them J1 Conn_01x05_Male, J10 Conn_01x01_Female, J11 Conn_01x01_Female, J2 Conn_01x05_Female, J3 Conn_01x01_Female, J4 Conn_01x01_Female, J5 Conn_01x01_Female, J6 Conn_01x01_Female, J7 Conn_01x02_Female, J8 Conn_01x01_Female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

Commit message: updated
Parts:
- moved J10 3.31 mm to (147.4, 121.3)
- moved J11 3.31 mm to (147.4, 116.7)
- moved J8 3.31 mm to (141.8, 121.3)
- moved J9 3.31 mm to (141.8, 116.7)
- moved J3 3.31 mm to (132.1, 116.7)
- moved J4 3.31 mm to (132.1, 121.3)
- moved J5 3.31 mm to (137.7, 116.7)
- moved J6 3.31 mm to (137.6, 121.3)
