File: joycon-board/joycon/joycon/joycon.kicad_pcb (KiCad board)
At the start: 2 copper layers, 21.6 x 20 mm, 11 parts, among them J1 Conn_01x05_Male, J10 Conn_01x01_Female, J11 Conn_01x01_Female, J2 Conn_01x05_Female, J3 Conn_01x01_Female, J4 Conn_01x01_Female, J5 Conn_01x01_Female, J6 Conn_01x01_Female, J7 Conn_01x02_Female, J8 Conn_01x01_Female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

Commit message: joystick-PCB
Parts:
- removed J10, J11, J4, J5, J6: Conn_01x01_Female, Connector_PinSocket_1.27mm:PinSocket_1x01_P1.27mm_Vertical
- added REF**: MountingHole_2.1mm, MountingHole:MountingHole_2.1mm, F.Cu at (148.2, 89.5)
- added REF**: MountingHole_2.1mm, MountingHole:MountingHole_2.1mm, F.Cu at (131.1, 105.0)
- J3: value Conn_01x01_Female -> Conn_01x03_Female; footprint Connector_PinSocket_1.27mm:PinSocket_1x01_P1.27mm_Vertical -> Connector_PinSocket_2.54mm:PinSocket_1x03_P2.54mm_Vertical
- J8, J9: value Conn_01x01_Female -> Conn_01x02_Female; footprint Connector_PinSocket_1.27mm:PinSocket_1x01_P1.27mm_Vertical -> Connector_PinSocket_2.54mm:PinSocket_1x02_P2.54mm_Vertical
- moved J3 26.4 mm to (142.5, 89.2), turned to -90 degrees
- moved J7 17.8 mm to (148.4, 102.7), turned to 0 degrees
- moved J8 13.1 mm to (144.7, 105.2), turned to -90 degrees
- moved J9 8.84 mm to (138.3, 105.2), turned to -90 degrees
Connections:
- J3 pad 1: unconnected-(J3-Pad1) -> Net-(J7-Pad1)
- J7 pad 1: Net-(J5-Pad1) -> Net-(J7-Pad1)
- J7 pad 2: Net-(J11-Pad1) -> GND
- J8 pad 1: Net-(J1-Pad1) -> Net-(J8-Pad1)
- J9 pad 1: unconnected-(J9-Pad1) -> Net-(J9-Pad1)
Routing:
- net GND: track 10.1 -> 54.8 mm
- net Net-(J8-Pad1): track 0.00 -> 17.9 mm
- net Net-(J1-Pad1): track 2.83 -> 20.1 mm
- net Net-(J9-Pad1): track 0.00 -> 16.3 mm
- net Net-(J7-Pad1): track 0.00 -> 15.9 mm
- net Net-(J1-Pad2): track 5.29 -> 19.1 mm
- net Net-(J1-Pad3): track 7.75 -> 18.9 mm
- net Net-(J1-Pad5): track 12.1 -> 17.9 mm
Other:
- outline, holes or cut-outs redrawn
- board text added: "B1"
- board text added: "B2"
- board text added: "B3"
