File: joycon-board/joycon/joycon/joycon.kicad_sch (KiCad schematic)
At the start: 2 parts, among them J1 Conn_01x05_Male, J2 Conn_01x05_Female

Commit message: updated
Parts:
- added J10, J11, J3, J4, J5, J6, J8, J9: Conn_01x01_Female, Connector_PinSocket_1.27mm:PinSocket_1x01_P1.27mm_Vertical, symbol Connector:Conn_01x01_Female
- added J7: Conn_01x02_Female, Connector_PinSocket_2.54mm:PinSocket_1x02_P2.54mm_Vertical, symbol Connector:Conn_01x02_Female
Connections:
- net GND: now also J10.1 (Pin_1), J6.1 (Pin_1)
- net at J1.1 (Pin_1), J2.1 (Pin_1): now also J4.1 (Pin_1), J8.1 (Pin_1)
- new net: J5.1 (Pin_1), J7.1 (Pin_1)
- new net: J11.1 (Pin_1), J7.2 (Pin_2)
Other:
- note added: "GND"
- note added: "VDD"
- moved on the sheet: J1, J2

Commit message: joystick-PCB
Parts:
- removed J10, J11, J3, J4, J5, J6, J8, J9: Conn_01x01_Female, Connector_PinSocket_1.27mm:PinSocket_1x01_P1.27mm_Vertical, symbol Connector:Conn_01x01_Female
- added J3: Conn_01x03_Female, Connector_PinSocket_2.54mm:PinSocket_1x03_P2.54mm_Vertical, symbol Connector:Conn_01x03_Female
- added J8, J9: Conn_01x02_Female, Connector_PinSocket_2.54mm:PinSocket_1x02_P2.54mm_Vertical, symbol Connector:Conn_01x02_Female
Connections:
- net GND: now also J7.2 (Pin_2), J8.2 (Pin_2), J9.2 (Pin_2)
- net at J7.1 (Pin_1): now also J3.1 (Pin_1)
- new net: J3.2 (Pin_2), J8.1 (Pin_1)
- new net: J3.3 (Pin_3), J9.1 (Pin_1)
