File: board/lower_v3.kicad_pcb (KiCad board)
At the start: 2 copper layers, 39.6 x 59.9 mm, 21 parts, among them J1 POWER, J10 PIN_RING_MOTOR, J11 PIN_PINKY_MOTOR, J12 PIN_PINKY_SPLAY, J13 PIN_RING_SPLAY, J14 PIN_MIDDLE_SPLAY, J15 PIN_INDEX_SPLAY, J16 PIN_THUMB_SPLAY, J19 Conn_01x08_Male, J2 PIN_PINKY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

Commit message: Remove via
Routing:
- net Net-(J19-Pad5): track 52.4 -> 50.3 mm, vias 1 -> 0
- net Net-(J19-Pad3): track 57.4 -> 55.7 mm
- net Net-(J19-Pad6): track 51.6 -> 50.1 mm
Changed lines of the file:
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@@
   (segment (start 145.138755 95.251245) (end 142.24 98.15) (width 0.25) (layer "F.Cu") (net 13))
   (segment (start 146.05 95.251245) (end 145.138755 95.251245) (width 0.25) (layer "F.Cu") (net 13))
-  (segment (start 139.7 67.925) (end 138.525 69.1) (width 0.25) (layer "F.Cu") (net 14))
-  (segment (start 138.525 69.1) (end 138.525 71.025) (width 0.25) (layer "F.Cu") (net 14))
-  (segment (start 138.525 71.025) (end 133.862299 75.687701) (width 0.25) (layer "F.Cu") (net 14))
-  (via (at 133.862299 75.687701) (size 0.8) (drill 0.4) (layers "F.Cu" "B.Cu") (free) (net 14))
-  (segment (start 135.81 97.590812) (end 135.81 77.644) (width 0.25) (layer "B.Cu") (net 14))
-  (segment (start 116.84 110.85) (end 122.550812 110.85) (width 0.25) (layer "B.Cu") (net 14))
-  (segment (start 133.862299 75.696299) (end 133.862299 75.687701) (width 0.25) (layer "B.Cu") (net 14))
-  (segment (start 135.81 77.644) (end 133.862299 75.696299) (width 0.25) (layer "B.Cu") (net 14))
-  (segment (start 122.550812 110.85) (end 135.81 97.590812) (width 0.25) (layer "B.Cu") (net 14))
-  (segment (start 134.62 72.39) (end 132.08 74.93) (width 0.25) (layer "F.Cu") (net 15))
-  (segment (start 134.62 70.465) (end 134.62 72.39) (width 0.25) (layer "F.Cu") (net 15))
-  (via (at 132.08 74.93) (size 0.8) (drill 0.4) (layers "F.Cu" "B.Cu") (net 15))
-  (segment (start 132.08 74.93) (end 135.36 78.21) (width 0.25) (layer "B.Cu") (net 15))
+  (segment (start 138.43 72.63261) (end 138.43 69.195) (width 0.25) (layer "F.Cu") (net 14))
+  (segment (start 137.408305 73.654305) (end 138.43 72.63261) (width 0.25) (layer "F.Cu") (net 14))
+  (segment (start 138.43 69.195) (end 139.7 67.925) (width 0.25) (layer "F.Cu") (net 14))
+  (via (at 137.408305 73.654305) (size 0.8) (drill 0.4) (layers "F.Cu" "B.Cu") (free) (net 14))
+  (segment (start 137.408305 73.654305) (end 136.398 74.66461) (width 0.25) (layer "B.Cu") (net 14))
+  (segment (start 135.81 75.264) (end 135.81 97.590812) (width 0.25) (layer "B.Cu") (net 14))
+  (segment (start 136.398 74.66461) (end 136.398 74.676) (width 0.25) (layer "B.Cu") (net 14))
+  (segment (start 135.81 97.590812) (end 122.550812 110.85) (width 0.25) (layer "B.Cu") (net 14))
+  (segment (start 122.550812 110.85) (end 116.84 110.85) (width 0.25) (layer "B.Cu") (net 14))
+  (segment (start 136.398 74.676) (end 135.81 75.264) (width 0.25) (layer "B.Cu") (net 14))
+  (segment (start 135.36 71.205) (end 135.36 97.404416) (width 0.25) (layer "B.Cu") (net 15))
+  (segment (start 134.62 70.465) (end 135.36 71.205) (width 0.25) (layer "B.Cu") (net 15))
   (segment (start 124.454416 108.31) (end 116.84 108.31) (width 0.25) (layer "B.Cu") (net 15))
-  (segment (start 135.36 78.21) (end 135.36 97.404416) (width 0.25) (layer "B.Cu") (net 15))
   (segment (start 135.36 97.404416) (end 124.454416 108.31) (width 0.25) (layer "B.Cu") (net 15))
   (segment (start 137.157208 88) (end 137.9 87.257208) (width 0.25) (layer "F.Cu") (net 17))
@@
   (segment (start 142.24 93.07) (end 144.018 91.292) (width 0.25) (layer "F.Cu") (net 18))
   (segment (start 136.26 75.827208) (end 136.26 97.777208) (width 0.25) (layer "B.Cu") (net 19))
+  (segment (start 138.43 73.657208) (end 137.412604 74.674604) (width 0.25) (layer "B.Cu") (net 19))
   (segment (start 137.414 74.673208) (end 136.26 75.827208) (width 0.25) (layer "B.Cu") (net 19))
-  (segment (start 137.16 67.925) (end 138.335 69.1) (width 0.25) (layer "B.Cu") (net 19))
-  (segment (start 138.335 73.752208) (end 137.412604 74.674604) (width 0.25) (layer "B.Cu") (net 19))
+  (segment (start 138.43 69.195) (end 138.43 73.657208) (width 0.25) (layer "B.Cu") (net 19))
   (segment (start 120.647208 113.39) (end 116.84 113.39) (width 0.25) (layer "B.Cu") (net 19))
-  (segment (start 138.335 69.1) (end 138.335 73.752208) (width 0.25) (layer "B.Cu") (net 19))
+  (segment (start 137.16 67.925) (end 138.43 69.195) (width 0.25) (layer "B.Cu") (net 19))
   (segment (start 136.26 97.777208) (end 120.647208 113.39) (width 0.25) (layer "B.Cu") (net 19))
-  (segment (start 137.16 70.465) (end 137.16 71.12) (width 0.25) (layer "F.Cu") (net 20))
-  (segment (start 132.08 76.2) (end 134.17 74.11) (width 0.25) (layer "F.Cu") (net 20))
-  (segment (start 137.16 71.12) (end 134.17 74.11) (width 0.25) (layer "F.Cu") (net 20))
-  (via (at 132.08 76.2) (size 0.8) (drill 0.4) (layers "F.Cu" "B.Cu") (net 20))
-  (segment (start 116.84 105.77) (end 126.35802 105.77) (width 0.25) (layer "B.Cu") (net 20))
-  (segment (start 126.35802 105.77) (end 134.91 97.21802) (width 0.25) (layer "B.Cu") (net 20))
-  (segment (start 134.91 79.03) (end 132.08 76.2) (width 0.25) (layer "B.Cu") (net 20))
-  (segment (start 134.91 97.21802) (end 134.91 79.03) (width 0.25) (layer "B.Cu") (net 20))
+  (segment (start 134.366 72.644) (end 136.545 70.465) (width 0.25) (layer "F.Cu") (net 20))
+  (segment (start 136.545 70.465) (end 137.16 70.465) (width 0.25) (layer "F.Cu") (net 20))
+  (segment (start 134.366 73.66) (end 134.366 72.644) (width 0.25) (layer "F.Cu") (net 20))
+  (via (at 134.366 73.66) (size 0.8) (drill 0.4) (layers "F.Cu" "B.Cu") (net 20))
+  (segment (start 134.91 74.204) (end 134.91 97.21802) (width 0.25) (layer "B.Cu") (net 20))
+  (segment (start 134.91 97.21802) (end 126.35802 105.77) (width 0.25) (layer "B.Cu") (net 20))
+  (segment (start 126.35802 105.77) (end 116.84 105.77) (width 0.25) (layer "B.Cu") (net 20))
+  (segment (start 134.366 73.66) (end 134.91 74.204) (width 0.25) (layer "B.Cu") (net 20))
   (segment (start 120.833604 113.84) (end 118.57 113.84) (width 0.25) (layer "B.Cu") (net 21))
   (segment (start 139.065 73.66) (end 139.063604 73.66) (width 0.25) (layer "B.Cu") (net 21))
